Commit message: wip

File: assets/robots/flamingo_edu/urdf/Edu_v4.urdf (robot description, URDF)
Before this commit: robot Edu_v4, 9 links, 8 joints
Links:
- link base_link: geometry collision mesh filename=base_link.STL; visual mesh filename=base_link.STL
- link front_cover_link: geometry collision mesh filename=front_cover_link.STL; visual mesh filename=front_cover_link.STL
- link left_leg_link: geometry collision mesh filename=left_leg_link.STL; visual mesh filename=left_leg_link.STL
- link left_shoulder_link: geometry collision mesh filename=left_shoulder_link.STL; visual mesh filename=left_shoulder_link.STL
- link left_wheel_link: geometry collision mesh filename=left_wheel_link.STL; visual mesh filename=left_wheel_link.STL
- link rear_cover_link: geometry collision mesh filename=rear_cover_link.STL; visual mesh filename=rear_cover_link.STL
- link right_leg_link: geometry collision mesh filename=right_leg_link.STL; visual mesh filename=right_leg_link.STL
- link right_shoulder_link: geometry collision mesh filename=right_shoulder_link.STL; visual mesh filename=right_shoulder_link.STL
- link right_wheel_link: geometry collision mesh filename=right_wheel_link.STL; visual mesh filename=right_wheel_link.STL
