Commit message: support for markers for event causality

File: assets/robots/rover/m2020.urdf (robot description, URDF)
Before this commit: robot Perseverance, 115 links, 114 joints
Links:
- removed link ground
- link Body_BogieLeft: mass 0 -> 1; geometry visual mesh filename=Left_Bogie.stl scale=1 1 1
- link Body_BogieRight: mass 0 -> 1; geometry visual mesh filename=Right_Bogie.stl scale=1 1 1
- link Body_Chassis: mass 0 -> 1; geometry visual mesh filename=CHASSIS.stl scale=1 1 1
- link Body_CorerFeed: mass 0 -> 1; geometry visual mesh filename=AbradingBitInTurretAtZeroFeed.stl scale=1 1 1
- link Body_Differential: mass 0 -> 1; geometry visual mesh filename=CenterDifferential.stl scale=1 1 1
- link Body_HGA_AZ: mass 0 -> 1; geometry visual mesh filename=HGA_AZ.stl scale=1 1 1
- link Body_HGA_EL: mass 0 -> 1; geometry visual mesh filename=HGA_EL.stl scale=1 1 1
- link Body_MHS_DebrisShield: mass 0 -> 1
- link Body_RA_Base: mass 0 -> 1
- link Body_RA_Link1: mass 0 -> 1; geometry visual mesh filename=Arm_LINK_1.stl scale=1 1 1
- link Body_RA_Link2: mass 0 -> 1; geometry visual mesh filename=Arm_LINK_2.stl scale=1 1 1
- link Body_RA_Link3: mass 0 -> 1; geometry visual mesh filename=Arm_LINK_3.stl scale=1 1 1
- link Body_RA_Link4: mass 0 -> 1; geometry visual mesh filename=Arm_LINK_4.stl scale=1 1 1
- link Body_RA_Link5: mass 0 -> 1; geometry visual mesh filename=Arm_LINK_5.stl scale=1 1 1
- link Body_RSM_AZ: mass 0 -> 1; geometry visual mesh filename=RSM.stl scale=1 1 1
- link Body_RSM_EL: mass 0 -> 1; geometry visual mesh filename=RSM_Head.stl scale=1 1 1
- link Body_RockerLeft: mass 0 -> 1; geometry visual mesh filename=Left_Rocker.stl scale=1 1 1
- link Body_RockerRight: mass 0 -> 1; geometry visual mesh filename=Right_Rocker.stl scale=1 1 1
- link Body_SHERLOC_Cap: mass 0 -> 1; geometry visual mesh filename=ContextImager_Cap.stl scale=1 1 1
- link Body_StabilizerFar: mass 0 -> 1; geometry visual mesh filename=StabilizerFarInTurret.stl scale=1 1 1
- link Body_StabilizerNear: mass 0 -> 1; geometry visual mesh filename=StabilizerNearInTurret.stl scale=1 1 1
- link Body_SteerLeftFront: mass 0 -> 1; geometry visual mesh filename=Steer_LeftFront.stl scale=1 1 1
- link Body_SteerLeftRear: mass 0 -> 1; geometry visual mesh filename=Steer_LeftRear.stl scale=1 1 1
- link Body_SteerRightFront: mass 0 -> 1; geometry visual mesh filename=Steer_RightFront.stl scale=1 1 1
- link Body_SteerRightRear: mass 0 -> 1; geometry visual mesh filename=Steer_RightRear.stl scale=1 1 1
- link Body_Turret: mass 0 -> 1; geometry visual mesh filename=Turret.stl scale=1 1 1
- link Body_WATSON_Cap: mass 0 -> 1; geometry visual mesh filename=WATSON_Camera_Cap.stl scale=1 1 1
- link Body_WheelLeftFront: mass 0 -> 1; geometry visual mesh filename=Wheel_LeftFront.stl scale=1 1 1
- link Body_WheelLeftMiddle: mass 0 -> 1; geometry visual mesh filename=Wheel_LeftMiddle.stl scale=1 1 1
- link Body_WheelLeftRear: mass 0 -> 1; geometry visual mesh filename=Wheel_LeftRear.stl scale=1 1 1
- link Body_WheelRightFront: mass 0 -> 1; geometry visual mesh filename=Wheel_RightFront.stl scale=1 1 1
- link Body_WheelRightMiddle: mass 0 -> 1; geometry visual mesh filename=Wheel_RightMiddle.stl scale=1 1 1
- link Body_WheelRightRear: mass 0 -> 1; geometry visual mesh filename=Wheel_RightRear.stl scale=1 1 1
- link Frame_ANT: mass 0 -> 1
- link Frame_ATS1: mass 0 -> 1
- link Frame_ATS2: mass 0 -> 1
- link Frame_ATS3: mass 0 -> 1
- link Frame_ATS4: mass 0 -> 1
- link Frame_ATS5: mass 0 -> 1
- link Frame_BOGIE_L: mass 0 -> 1
- link Frame_BOGIE_R: mass 0 -> 1
- link Frame_CAL_MC1: mass 0 -> 1
- link Frame_CAL_MC2: mass 0 -> 1
- link Frame_CAL_PIXL: mass 0 -> 1
- link Frame_CAL_SC: mass 0 -> 1
- link Frame_CAL_SHERLOC: mass 0 -> 1
- link Frame_DIFF: mass 0 -> 1
- link Frame_DOCKING_POST: mass 0 -> 1
- link Frame_DRILL: mass 0 -> 1
- link Frame_FCS: mass 0 -> 1
- link Frame_FHC1: mass 0 -> 1
- link Frame_FHC1_FOV: mass 0 -> 1
- link Frame_FHC2: mass 0 -> 1
- link Frame_FHC2_FOV: mass 0 -> 1
- link Frame_FHC3: mass 0 -> 1
- link Frame_FHC3_FOV: mass 0 -> 1
- link Frame_FHC4: mass 0 -> 1
- link Frame_FHC4_FOV: mass 0 -> 1
- link Frame_FHCB: mass 0 -> 1
- link Frame_GDRT: mass 0 -> 1
- link Frame_HGAG: mass 0 -> 1
- link Frame_HGAS: mass 0 -> 1
- link Frame_HS: mass 0 -> 1
- link Frame_ICU: mass 0 -> 1
- link Frame_MAZ: mass 0 -> 1
- link Frame_MCL: mass 0 -> 1
- link Frame_MCR: mass 0 -> 1
- link Frame_MEL: mass 0 -> 1
- link Frame_MI: mass 0 -> 1
- link Frame_MOXIE: mass 0 -> 1
- link Frame_NCL: mass 0 -> 1
- link Frame_NCL_FOV: mass 0 -> 1
- link Frame_NCR: mass 0 -> 1
- link Frame_NCR_FOV: mass 0 -> 1
- link Frame_PIXL: mass 0 -> 1
- link Frame_RA1: mass 0 -> 1
- link Frame_RA2: mass 0 -> 1
- link Frame_RA3: mass 0 -> 1
- link Frame_RA4: mass 0 -> 1
- link Frame_RA5: mass 0 -> 1
- link Frame_RA6: mass 0 -> 1
- link Frame_RA_BASE: mass 0 -> 1
- link Frame_RDS: mass 0 -> 1
- link Frame_RHC1: mass 0 -> 1
- link Frame_RHC1_FOV: mass 0 -> 1
- link Frame_RHC2: mass 0 -> 1
- link Frame_RHC2_FOV: mass 0 -> 1
- link Frame_RIMFAX: mass 0 -> 1
- link Frame_RIMUA: mass 0 -> 1
- link Frame_RIMUB: mass 0 -> 1
- link Frame_RMECH: mass 0 -> 1
- link Frame_RNAV: mass 0 -> 1
- link Frame_ROCKER_L: mass 0 -> 1
- link Frame_ROCKER_R: mass 0 -> 1
- link Frame_SCI: mass 0 -> 1
- link Frame_SCIR: mass 0 -> 1
- link Frame_SCLIBS: mass 0 -> 1
- link Frame_SCRMI: mass 0 -> 1
- link Frame_SHERLOC: mass 0 -> 1
- link Frame_STEER_LF: mass 0 -> 1
- link Frame_STEER_LR: mass 0 -> 1
- link Frame_STEER_RF: mass 0 -> 1
- link Frame_STEER_RR: mass 0 -> 1
- link Frame_TIRS: mass 0 -> 1
- link Frame_TURRET: mass 0 -> 1
- link Frame_WATSON: mass 0 -> 1
- link Frame_WHEEL_LF: mass 0 -> 1
- link Frame_WHEEL_LM: mass 0 -> 1
- link Frame_WHEEL_LR: mass 0 -> 1
- link Frame_WHEEL_RF: mass 0 -> 1
- link Frame_WHEEL_RM: mass 0 -> 1
- link Frame_WHEEL_RR: mass 0 -> 1
- link Frame_WS1: mass 0 -> 1
- link Frame_WS2: mass 0 -> 1
Joints:
- removed joint JointRoot
