Commit message: so-arm 101 initial rendering bug isolated

File: assets/manipulators/so-101/so101_new_calib.urdf (robot description, URDF)
Before this commit: robot so101_new_calib, 8 links, 7 joints
Joints:
- joint shoulder_pan: limit lower=-1.91986 upper=1.91986 effort=10 velocity=10 -> lower=-7 upper=0 effort=10 velocity=10

Commit message: wip so-arm101

File: assets/manipulators/so-101/so101_new_calib.urdf (robot description, URDF)
Before this commit: robot so101_new_calib, 8 links, 7 joints
Joints:
- joint shoulder_pan: limit lower=-7 upper=0 effort=10 velocity=10 -> lower=-1.91986 upper=1.91986 effort=10 velocity=10

Commit message: joint fix

File: assets/manipulators/so-101/so101_new_calib.urdf (robot description, URDF)
Before this commit: robot so101_new_calib, 8 links, 7 joints
Joints:
- joint shoulder_pan: limit lower=-1.91986 upper=1.91986 effort=10 velocity=10 -> lower=-5.91986 upper=5.91986 effort=10 velocity=10
